Commit message: lauch file added

File: description/robot_core.xacro (robot description, xacro)
@@ -1,5 +1,5 @@
 <?xml version="1.0"?>
 <robot xmlns:xacro="http://www.ros.org/wiki/xacro">
-    <xacro:include filename="/home/ajay_stark/Documents/ros/articubot_one/dev_ws/src/articubot_one/description/inertial_macros.xacro"/>
+    <xacro:include filename="/home/i-corinthian/Documents/ros/articubot/ros_ws/src/articubot_one/description/inertial_macros.xacro"/>
     <material name="White">
         <color rgba="1 1 1 1"/>
@@ -40,4 +40,7 @@
     </xacro:inertial_box>
     </link>
+    <gazebo reference="chassis">
+        <material>Gazebo/White</material>
+    </gazebo>
     <!-- LEFT WHEEL -->
     <joint name="left_wheel_joint" type="continuous">
@@ -63,4 +66,7 @@
         </xacro:inertial_cylinder>
     </link>
+    <gazebo reference="left_wheel">
+        <material>Gazebo/Blue</material>
+    </gazebo>
     <!-- RIGHT WHEEL -->
     <joint name="right_wheel_joint" type="continuous">
@@ -86,4 +92,7 @@
         </xacro:inertial_cylinder>
     </link>
+    <gazebo reference="right_wheel">
+        <material>Gazebo/Blue</material>
+    </gazebo>
     <!-- CASER WHEEL-->
     <joint name="caser_wheel_joint" type="fixed">
@@ -108,3 +117,6 @@
         </xacro:inertial_sphere>
     </link>
+    <gazebo reference="caster_wheel">
+        <material>Gazebo/Black</material>
+    </gazebo>
 </robot>
